File: Full_96/PCB/Keyboard.sch (KiCad schematic (older format))
At the start: 207 parts, among them J1 Battery, SW1 SW_DIP_x01, U1 TinyPICO_Nano

Commit message: Libraries moved to global location, layout started for Full_75
Parts:
- MX1, MX10, MX11, MX12, MX13, MX14, MX15, MX16, MX17, MX18, MX19, MX2, MX20, MX21, MX22, MX23, MX24, MX25, MX26, MX27, MX28, MX29, MX3, MX30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: symbol MX_Alps_Hybrid:MX-NoLED -> _MX_Alps_Hybrid:MX-NoLED
- U1: symbol TinyPICO_Nano:TinyPICO_Nano -> _MCU_Devboards:TinyPICO_Nano
- USB1: symbol Type-C:USB4085-GF-A -> _Connectors:USB4085-GF-A-Type-C
