File: Full_75/Full_75/Full_75.sch (KiCad schematic (older format))
At the start: 185 parts, among them J1 Battery, J2 Numpad_PWR, SW1 SW_DIP_x01, U1 TinyPICO_Nano, U2 MIC4801, U3 MIC4801, U4 MIC4801, U5 MIC4801, U6 MIC4801

Commit message: finished 75% layout
Parts:
- J2: footprint _Connectors:01x02_MillMax_Springloaded_Pin -> _Connectors:01x03_MillMax_Springloaded_Pin; symbol Connector_Generic:Conn_01x02 -> Connector_Generic:Conn_01x03
Connections:
- net +5V: now also D1.2 (A), D2.2 (A), D3.2 (A), D4.2 (A), J2.1 (Pin_1); no longer J2.2 (Pin_2)
- net Col[0]: now also U1.12 (D18); no longer U1.24 (D38)
- net Col[10]: now also U1.32 (D41); no longer U1.19 (D12)
- net Col[11]: now also U1.23 (D36); no longer U1.25 (D35)
- net Col[12]: now also U1.24 (D38); no longer MX93.1 (COL), U1.26 (D34)
- net Col[13]: now also MX93.1 (COL), U1.25 (D35); no longer U1.27 (D39)
- net Col[1]: now also U1.13 (D20); no longer U1.23 (D36)
- net Col[2]: now also U1.14 (D17); no longer U1.10 (D22)
- net Col[3]: now also U1.15 (D21); no longer U1.11 (D24)
- net Col[4]: now also U1.16 (D16); no longer U1.12 (D18)
- net Col[5]: now also U1.17 (D15); no longer U1.13 (D20)
- net Col[6]: now also U1.18 (D14); no longer MX62.1 (COL), U1.15 (D21)
- net Col[7]: now also MX62.1 (COL), U1.19 (D12); no longer U1.16 (D16)
- net Col[8]: now also U1.20 (D13); no longer U1.17 (D15)
- net Col[9]: now also U1.26 (D34); no longer U1.18 (D14)
- net GND: now also J2.2 (Pin_2); no longer J2.1 (Pin_1)
- net LED_EN0: now also U1.31 (D40); no longer U1.28 (D42)
- net LED_EN1: now also U1.30 (D28); no longer U1.29 (D23)
- net LED_EN2: now also U1.29 (D23); no longer U1.30 (D28)
- net LED_EN3: now also U1.28 (D42); no longer U1.31 (D40)
- net LED_EN4: now also U1.27 (D39); no longer U1.14 (D17)
- net Row[0]: now also U1.21 (D10); no longer U1.22 (D11)
- net Row[1]: now also U1.11 (D24); no longer U1.32 (D41)
- new net LED_EN_NUM: J2.3 (Pin_3), U1.10 (D22)
- no-connect marks 6 -> 5
Other:
- moved on the sheet: D3, D4, D63, D94, MX62, MX93
