File: Full_75/Full_75/Full_75.kicad_pcb (KiCad board)
At the start: 2 copper layers, 285.7 x 114.3 mm, 185 parts, among them J1 Battery, J2 Numpad_PWR, SW1 SW_DIP_x01, U1 TinyPICO_Nano, U2 MIC4801, U3 MIC4801, U4 MIC4801, U5 MIC4801, U6 MIC4801

Commit message: finished 75% layout
Parts:
- added REF**: MountingHole_2.2mm_M2, MountingHole:MountingHole_2.2mm_M2, F.Cu at (101.6, 96.0)
- added REF**: MountingHole_2.2mm_M2, MountingHole:MountingHole_2.2mm_M2, F.Cu at (225.4, 115.1)
- added REF**: MountingHole_2.2mm_M2, MountingHole:MountingHole_2.2mm_M2, F.Cu at (277.8, 133.3)
- added REF**: MountingHole_2.2mm_M2, MountingHole:MountingHole_2.2mm_M2, F.Cu at (163.5, 38.9)
- added REF**: MountingHole_2.2mm_M2, MountingHole:MountingHole_2.2mm_M2, F.Cu at (68.3, 38.9)
- added REF**: MountingHole_2.2mm_M2, MountingHole:MountingHole_2.2mm_M2, F.Cu at (258.7, 38.9)
- added REF**: MountingHole_2.2mm_M2, MountingHole:MountingHole_2.2mm_M2, F.Cu at (192.1, 77.0)
- added REF**: MountingHole_2.2mm_M2, MountingHole:MountingHole_2.2mm_M2, F.Cu at (58.7, 77.0)
- added REF**: MountingHole_2.2mm_M2, MountingHole:MountingHole_2.2mm_M2, F.Cu at (273.0, 96.0)
- added REF**: MountingHole_2.2mm_M2, MountingHole:MountingHole_2.2mm_M2, F.Cu at (77.8, 134.1)
- added REF**: MountingHole_2.2mm_M2, MountingHole:MountingHole_2.2mm_M2, F.Cu at (149.2, 115.1)
- C2, C3, C4, C5, R4, R5, R6, R7, R8, U3, U4, U5, U6: moved to B.Cu
- J2: footprint _Connectors:01x02_MillMax_Springloaded_Pin -> _Connectors:01x03_MillMax_Springloaded_Pin
- moved R4 130.6 mm to (74.3, 116.5), turned to 180 degrees
- moved R8 116.6 mm to (295.3, 131.1)
- moved C5 107.7 mm to (298.8, 132.0), turned to 90 degrees
- moved U3 88.0 mm to (152.1, 126.1), turned to 90 degrees
- moved U6 83.4 mm to (296.9, 126.1), turned to 90 degrees
- moved R7 79.7 mm to (255.3, 131.1)
- moved C4 77.7 mm to (260.7, 129.4), turned to 90 degrees
- moved C3 57.8 mm to (218.1, 129.4), turned to 90 degrees
- moved R5 53.6 mm to (150.5, 131.1)
- moved U5 52.8 mm to (256.9, 126.1), turned to 90 degrees
- moved R6 36.5 mm to (212.8, 131.1)
- moved U4 36.1 mm to (214.3, 126.1), turned to 90 degrees
- moved C2 34.7 mm to (155.9, 129.4), turned to 90 degrees
- moved D62 19.0 mm to (177.8, 116.3)
- moved D68 19.0 mm to (196.8, 116.3)
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Connections:
- D1 pad 2: Net-(D1-Pad2) -> +5V
- D2 pad 2: Net-(D1-Pad2) -> +5V
- D3 pad 2: Net-(D3-Pad2) -> +5V
- D4 pad 2: Net-(D3-Pad2) -> +5V
- J2 pad 1: GND -> +5V
- J2 pad 2: +5V -> GND
- MX62 pad 1: /Col[6] -> /Col[7]
- MX93 pad 1: /Col[12] -> /Col[13]
- U1 pad 10: /Col[2] -> /LED_EN_NUM
- U1 pad 11: /Col[3] -> /Row[1]
- U1 pad 12: /Col[4] -> /Col[0]
- U1 pad 13: /Col[5] -> /Col[1]
- U1 pad 14: /LED_EN4 -> /Col[2]
- U1 pad 15: /Col[6] -> /Col[3]
- U1 pad 16: /Col[7] -> /Col[4]
- U1 pad 17: /Col[8] -> /Col[5]
- U1 pad 18: /Col[9] -> /Col[6]
- U1 pad 19: /Col[10] -> /Col[7]
- U1 pad 20: Net-(U1-Pad20) -> /Col[8]
- U1 pad 21: Net-(U1-Pad21) -> /Row[0]
- U1 pad 22: /Row[0] -> Net-(U1-Pad22)
- U1 pad 23: /Col[1] -> /Col[11]
- U1 pad 24: /Col[0] -> /Col[12]
- U1 pad 25: /Col[11] -> /Col[13]
- U1 pad 26: /Col[12] -> /Col[9]
- U1 pad 27: /Col[13] -> /LED_EN4
- U1 pad 28: /LED_EN0 -> /LED_EN3
- U1 pad 29: /LED_EN1 -> /LED_EN2
- U1 pad 30: /LED_EN2 -> /LED_EN1
- U1 pad 31: /LED_EN3 -> /LED_EN0
- U1 pad 32: /Row[1] -> /Col[10]
Routing:
- net /LED_CAT1: track 0.00 -> 439.1 mm, vias 0 -> 57
- net /LED_CAT2: track 0.00 -> 432.5 mm, vias 0 -> 55
- net /LED_CAT3: track 0.00 -> 385.6 mm, vias 0 -> 53
- net /LED_EN0: track 0.00 -> 373.8 mm, vias 0 -> 4
- net /Col[3]: track 0.00 -> 332.5 mm, vias 0 -> 1
- net /LED_EN_NUM: track 0.00 -> 291.4 mm, vias 0 -> 1
- net /Col[5]: track 0.00 -> 290.8 mm, vias 0 -> 1
- net /Col[4]: track 0.00 -> 288.8 mm, vias 0 -> 1
- net /LED_EN1: track 0.00 -> 280.2 mm, vias 0 -> 2
- net /LED_CAT4: track 0.00 -> 272.5 mm, vias 0 -> 35
- net /Col[0]: track 114.5 -> 386.8 mm, vias 0 -> 1
- net /Col[9]: track 0.00 -> 267.5 mm, vias 0 -> 3
- net /Col[7]: track 0.00 -> 251.8 mm, vias 0 -> 1
- net /Col[10]: track 0.00 -> 249.2 mm, vias 0 -> 3
- net /Col[1]: track 132.9 -> 382.1 mm, vias 0 -> 1
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Other:
- board outline removed
- rule trace_min: 0.2 -> 0

Commit message: LED code functional, working on switch matrix and profile storage
Parts:
- added G***: LOGO, _Silkscreens:YoRHa, F.Cu at (306.4, 109.9)
Other:
- board outline added: 285.7 x 118.3 mm
- board text added: "JLCJLCJLCJLC"
